File: PCB/WE MAKING IT TO ISEF WITH THIS ONE.kicad_sch (KiCad schematic)
At the start: 43 parts, among them IC1 ESP32-WROOM-32E-N16, J1 MSD-1-A - SD Card Read, J2 USB_C_Receptacle_USB2.0_16P, U1 ATSAMD51P20A-AUT, U2 AS7263-BLGT - Spectroscopy, U3 TPS546D24ARVFR - Step Down Tr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, U4 SST26VF016BT-104V/MF, Y1 Crystal, Y2 Crystal

Commit message: Add files via upload
Parts:
- removed Y2: Crystal, symbol Device:Crystal
- added C26, C27: C_US, actually dont hold me back capacitor:CAP_GCM18_1p7X0p9X0p9_MUR, symbol Device:C_US
- added Y3: Crystal, symbol Device:Crystal
Connections:
- net +3.3V: now also C19.1, C20.1, IC1.2 (3V3), R5.1
- net GNDD: now also C26.2, C27.2
- net GNDREF: now also C19.2, C20.2
- net at U2.11 (RX/SCL_S): now also IC1.12 (IO27), U1.71 (PC17), U3.3 (PMB_CLK), U3.39 (BCX_CLK)
- net at U2.12 (TX/SDA_S): now also IC1.11 (IO26), U1.70 (PC16), U3.2 (PMB_DATA), U3.40 (BCX_DAT)
- net at J1.CD: now also U1.122 (PB31)
- net at U1.1 (PA00): now also C26.1, Y3.1
- net at U1.2 (PA01): now also C27.1, Y3.2
Other:
- note added: "10k ohms^^"
- note added: "scl"
- note added: "sda"
- moved on the sheet: C10, C11, C12, C13, C14, C15, C16, C17, C18, C2, C3, C4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

Commit message: Add files via upload
Connections:
- net +3.3V: now also U2.14 (VDD2), U2.17 (VDD1)
Changed lines of the file:
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@@
 	)
 	(junction
+		(at 326.39 15.24)
+		(diameter 0)
+		(color 0 0 0 0)
+	)
+	(junction
 		(at 201.93 -213.36)
 		(diameter 0)
@@
 	(wire
 		(pts
+			(xy 326.39 10.16) (xy 326.39 15.24)
+		)
+		(stroke
+			(width 0)
+			(type default)
+		)
+	)
+	(wire
+		(pts
 			(xy 43.18 81.28) (xy 43.18 50.8)
 		)
@@
 					(unit 1)
 				)
+			)
+		)
+	)
+	(symbol
+		(lib_id "power:+3.3V")
+		(at 326.39 10.16 0)
+		(unit 1)
+		(body_style 1)
+		(exclude_from_sim no)
+		(in_bom yes)
+		(on_board yes)
+		(in_pos_files yes)
+		(dnp no)
+		(fields_autoplaced yes)
+		(property "Reference" "#PWR026"
+			(at 326.39 13.97 0)
+			(hide yes)
+			(show_name no)
+			(do_not_autoplace no)
+			(effects
+				(font
+					(size 1.27 1.27)
+				)
+			)
+		)
+		(property "Value" "+3.3V"
+			(at 326.39 5.08 0)
+			(show_name no)
+			(do_not_autoplace no)
+			(effects
+				(font
+					(size 1.27 1.27)
+				)
+			)
+		)
+		(property "Footprint" ""
+			(at 326.39 10.16 0)
+			(hide yes)
+			(show_name no)
+			(do_not_autoplace no)
+			(effects
+				(font
+					(size 1.27 1.27)
+				)
+			)
+		)
+		(property "Datasheet" ""
+			(at 326.39 10.16 0)
+			(hide yes)
+			(show_name no)
+			(do_not_autoplace no)
+			(effects
+				(font
+					(size 1.27 1.27)
+				)
+			)
+		)
+		(property "Description" "Power symbol creates a global label with name \"+3.3V\""
+			(at 326.39 10.16 0)
+			(hide yes)
+			(show_name no)
+			(do_not_autoplace no)
+			(effects
+				(font
+					(size 1.27 1.27)
+				)
+			)
+		)
+		(pin "1"
+		)
+		(instances
+			(project "WE MAKING IT TO ISEF WITH THIS ONE"
+				(path "/ab9c9e90-16c1-4fff-8322-fda1cac8bed0"
+					(reference "#PWR026")
+					(unit 1)
+				)

Commit message: Add files via upload
Parts:
- removed U3: TPS546D24ARVFR - Step Down Transformer, 12Vto5Vfootprint:RVF0040A, symbol 12Vto5V:TPS546D24ARVFR
- added JP2: SolderJumper_2_Bridged, symbol Jumper:SolderJumper_2_Bridged
Connections:
- net +3.3V: now also LED1.2
- net GNDD: now also U2.16 (GND), JP2.2 (B); no longer LED1.1
- net at U2.13 (~{INT}): now also U1.10 (PA03)
- net at U2.15 (LED_DRV): now also LED1.1; no longer LED1.2
- net at U2.2 (~{RESN}): now also U1.9 (PA02)
- net at IC1.25 (IO0): now also JP2.1 (A)
Other:
- note added: "0.1 microfarads^^"
- note added: "1 microfarads^^"
- note added: "10 microfarads^^"
- note added: "12 picofarads^^"
- note added: "22 microfarads^^"
- note added: "3a or 1a i havent decided yet"
- note removed: "0.1 picofarads^^"
- note removed: "1 picofarad^^"
- note removed: "10 picofarads^^"
- note removed: "40ma"
- moved on the sheet: C10, C11, C12, C13, C14, C15, C16, C17, C18, C2, C3, C4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

Commit message: Add files via upload
Connections:
- net Flash_Memory - Chip Select Line: now reaches U1.40 (PB11), U4.1 (CE#)
- net Flash_Memory - Serial Clock Line: now reaches U1.39 (PB10), U4.6 (SCK)
- net SCL Global Bus :D: now reaches U1.71 (PC17), U2.11 (RX/SCL_S)
- net SCL Global Bus :D: now also IC1.11 (IO26); no longer IC1.12 (IO27)
- net SDA Global Bus :D: now reaches U1.70 (PC16), U2.12 (TX/SDA_S)
- net SDA Global Bus :D: now also IC1.10 (IO25); no longer IC1.11 (IO26)
- net Spectroscopy Sensor - Interrupt Line: now reaches U1.10 (PA03), U2.13 (~{INT})
- net Spectroscopy Sensor - Reset Line: now reaches U1.9 (PA02), U2.2 (~{RESN})
- net Spectroscopy Sensor - I2C Enable Line: now reaches U1.21 (PA04), U2.8 (I2C_ENB)
- net SD_Card_Reader - CMD Line: now reaches J1.3 (CMD), U1.102 (PB26)
- net SD_Card_Reader - Clock Line: now reaches J1.5 (CLK), U1.103 (PB27)
- net USB-C - D- Line: now reaches J2.A7 (D-), J2.B7 (D-), U1.94 (PA24)
- net USB-C - D+ Line: now reaches J2.A6 (D+), J2.B6 (D+), U1.95 (PA25)
Other:
- note added: "9/9/26"
- note added: "Microplastic Detection PCB"
- note removed: "scl"
- note removed: "sda"
- moved on the sheet: C10, C11, C12, C13, C14, C15, C16, C17, C18, C19, C2, C20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
